File: electronics/kicad/antweight-controller-v2-2s/antweight-controller-v2-2s.kicad_pcb (KiCad board)
At the start: 2 copper layers, 100 x 100 mm, 30 parts, among them J10 3V3 GND VBAT_SW, J4 FUSED 2S INPUT, J5 MOTOR LEFT, J6 MOTOR RIGHT, J8 ESP32 LEFT ALL PINS, J9 ESP32 RIGHT SIGNALS, M1 N20 6V 50:1 MOTOR LEFT, M2 N20 6V 50:1 MOTOR RIGHT, SW1 MAIN POWER, U1 ESP32-C3 SUPERMINI, U2 DRV8833, U3 MINI-360 MP2307DN 3V3

Commit message: chore: first commit for 2S PCB routing and label/render updates
Parts:
- removed EXP1: PROTO_10X04_2P54, PROTO_10X04_2P54
- removed EXP2, EXP3, EXP4, EXP5: PROTO_CORNER_4X04_2P54, PROTO_CORNER_4X04_2P54
- removed M1: N20 6V 50:1 MOTOR LEFT, N20_10X12_MECHANICAL_PROVISIONAL
- removed M2: N20 6V 50:1 MOTOR RIGHT, N20_10X12_MECHANICAL_PROVISIONAL
- moved C1_C2 12.0 mm to (108.0, 104.2), turned to 180 degrees
- moved MB3 3.00 mm to (72.5, 83.9)
- moved MB4 3.00 mm to (72.5, 111.9)
- moved MB5 3.00 mm to (113.0, 83.9)
- moved MB6 3.00 mm to (113.0, 111.9)
Routing:
- net PROTO_VPLUS: track 143.1 -> 0.00 mm
- net VBAT_SW: track 0.00 -> 98.0 mm, vias 0 -> 1
- net 3V3: track 0.00 -> 83.6 mm, vias 0 -> 1
- net AIN1_GPIO7: track 0.00 -> 46.0 mm
- net GND: track 0.00 -> 45.9 mm
- net AIN2_GPIO6: track 0.00 -> 44.8 mm
- net M1B: track 0.00 -> 33.1 mm
- net BIN2_GPIO10: track 0.00 -> 32.5 mm
- net M2B: track 0.00 -> 30.3 mm
- net BIN1_GPIO9: track 0.00 -> 28.2 mm
- net M2A: track 0.00 -> 26.1 mm
- net M1A: track 0.00 -> 23.9 mm
- added copper zone on B.Cu, net GND
Other:
- outline, holes or cut-outs redrawn
- board text added: "A1 M2"
- board text added: "A2 M2"
- board text added: "AUX PWR"
- board text added: "B+"
- board text added: "B1 M1"
- board text added: "B2 M1"
- board text added: "HDR L"
- board text added: "HDR R"
- board text added: "IN+"
- board text added: "MOTOR DRIVER"
- board text added: "MTR L"
- board text added: "MTR R"
- board text added: "PWR SW"
- board text removed: "+IN"
- board text removed: "A1"
- board text removed: "A2"
- board text removed: "B1"
- board text removed: "B2"
- board text removed: "BAT+"
- board text removed: "DRV8833"
- board text removed: "J8"
- board text removed: "J9"
- board text removed: "MOTOR L"
- board text removed: "MOTOR R"
- board text removed: "PWR AUX"
- board text removed: "SW1"
