File: electronics/kicad/antweight-controller-v2-2s/antweight-controller-v2-2s.kicad_pcb (KiCad board)
At the start: 2 copper layers, 100 x 100 mm, 23 parts, among them J10 3V3 GND VBAT_SW, J4 FUSED 2S INPUT, J5 MOTOR LEFT, J6 MOTOR RIGHT, J8 ESP32 LEFT ALL PINS, J9 ESP32 RIGHT SIGNALS, SW1 MAIN POWER, U1 ESP32-C3 SUPERMINI, U2 DRV8833, U3 MINI-360 MP2307DN 3V3

Commit message: chore(electronics): refine v2/v3 2S PCB routing and DRC fixes
Parts:
- removed MB2: MOUSE_BITE, MOUSE_BITE_5X0.5
- J4: value FUSED 2S INPUT -> 2S LiPo JST-XH; footprint BATTERY_SOLDER_PADS_5A -> JST_XH_BATTERY_2PIN
Routing:
- net GND: track 45.9 -> 49.8 mm
Other:
- board text added: "+"
- board text added: "-"
- board text removed: "B+"
