File: electronics/kicad/rein3/antweight-controller-v2.kicad_pcb (KiCad board)
At the start: 2 copper layers, 36 x 67 mm, 11 parts, among them J10 3V3 GND VBAT_SW, J4 BATTERY, J5 MOTOR LEFT, J6 MOTOR RIGHT, J8 ESP32 LEFT ALL PINS, J9 ESP32 RIGHT SIGNALS, SW1 MAIN POWER, U1 ESP32-C3 SUPERMINI, U2 DRV8833, U3 3V3 BUCK-BOOST

Commit message: Update docs and publish KiCad WIP state
Routing:
- net GND: track 50.1 -> 161.1 mm
- net 3V3: track 19.2 -> 122.1 mm
- net AIN2_GPIO6: track 2.54 -> 58.9 mm
- net VBAT_SW: track 45.3 -> 84.8 mm
- net BIN1_GPIO9: track 5.08 -> 43.0 mm
- net AIN1_GPIO7: track 2.54 -> 31.5 mm
Other:
- board size 36 x 67 mm -> 46 x 67 mm
- board text removed: "J8"
- board text removed: "J9"
