File: electronics/kicad/rein3-2s/rein-2s-controller.kicad_pcb (KiCad board)
At the start: 2 copper layers, 46 x 67 mm, 11 parts, among them J10 3V3 GND VBAT_SW, J4 BATTERY, J5 MOTOR LEFT, J6 MOTOR RIGHT, J8 ESP32 LEFT ALL PINS, J9 ESP32 RIGHT SIGNALS, SW1 MAIN POWER, U1 ESP32-C3 SUPERMINI, U2 DRV8833, U3 3V3 BUCK-BOOST

Commit message: Update KiCad board variants and logo placement
Parts:
- SW1: value MAIN POWER -> SW EXT VBAT_RAW/VBAT_SW; footprint SWITCH_VERIFY -> SWITCH_EXT_1X02
- U3: value 3V3 BUCK-BOOST -> EXT REG LOGIC VIN GND VOUT; footprint REGULATOR_VERIFY -> REGULATOR_EXT_1X03
- moved C1_C2 14.6 mm to (53.0, 68.5), turned to -90 degrees
- moved U3 4.21 mm to (27.0, 68.5)
- moved SW1 2.50 mm to (22.2, 76.5)
- moved J4 2.00 mm to (34.5, 76.5)
Routing:
- net GND: track 161.6 -> 102.7 mm, vias 0 -> 1
- net 3V3: track 122.1 -> 93.9 mm
- net VBAT_SW: track 84.8 -> 74.6 mm
- net AIN1_GPIO7: track 31.5 -> 36.2 mm
- net VBAT_RAW: track 16.8 -> 18.0 mm
Other:
- board text added: "+8v"
- board text added: "BYPASS"
- board text added: "SW EXT"
- board text removed: "MAIN SW"
- board text removed: "MOTOR L"
- board text removed: "MOTOR R"
- board text removed: "OUT"
