File: electronics/kicad/hsd-antweight-2s-pcb/rein-2s-controller.kicad_sch (KiCad schematic)
At the start: 13 parts, among them J1 ESP32-C3_LEFT, J10 ACCESSORY_POWER, J2 ESP32-C3_RIGHT, J3 DRV8833_BREAKOUT, J4 BATTERY_1S, J5 MOTOR_LEFT, J6 MOTOR_RIGHT, J7 3V3_BUCK_BOOST, J8 ESP32_LEFT_ALL_PINS_BREAKOUT, J9 ESP32_RIGHT_BREAKOUT, SW1 MAIN_POWER

Commit message: docs(electronics): migrate remaining refs to 2S and add assembled renders
Parts:
- J4: value BATTERY_1S -> BATTERY_2S_7V4
Changed lines of the file:
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@@
 			)
 		)
-		(property "Value" "BATTERY_1S"
+		(property "Value" "BATTERY_2S_7V4"
 			(at 223.012 64.7446 0)
 			(effects
