File: electronics/kicad/hsd-antweight-2s-v2/hsd-antweight-2s-v3.kicad_pcb (KiCad board)
At the start: 2 copper layers, 78 x 56 mm, 10 parts, among them J10 3V3 GND VLIPO, J4 BATTERY, J5 MOTOR LEFT, J6 MOTOR RIGHT, SW1 SW EXT VBAT_RAW/VBAT_SW, U1 ESP32-C3 SUPERMINI, U2 DRV8833, U3 EXT REG LOGIC VIN GND VOUT

Commit message: v3: add render variants and restore clean pcb state
Other:
- board text added: "ON/OFF"
- board text removed: "SW EXT"
Changed lines of the file:
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@@
+		)
+	)
+	(gr_text "ON/OFF"
+		(at 80 43 0)
+		(layer "F.SilkS")
+		(effects
+			(font
+				(size 0.8 0.8)
+				(thickness 0.12)
+			)
 		)
 	)
@@
 		)
 	)
-	(gr_text "SW EXT"
-		(at 80 43 0)
-		(layer "B.SilkS")
-		(effects
-			(font
-				(size 0.8 0.8)
-				(thickness 0.12)
-			)
-			(justify mirror)
-		)
-	)
 	(gr_text "BYPASS"
 		(at 82 38.5 0)
@@
 	)
 	(gr_text "ROBOKTOBER.NL"
-		(at 58 82.5 0)
-		(layer "B.SilkS")
-		(effects
+		(at 57.5 80 0)
+		(layer "B.SilkS")
+		(effects
