File: electronics/kicad/hsd-antweight-2s-v3-fix/hsd-antweight-2s-v3.kicad_pcb (KiCad board)
At the start: 2 copper layers, 78 x 56 mm, 10 parts, among them J10 5V(3.7-5V) GND VLIPO, J4 BATTERY, J5 MOTOR LEFT, J6 MOTOR RIGHT, SW1 SW EXT VBAT_RAW/VBAT_SW, U1 ESP32-C3 SUPERMINI, U2 DRV8833, U3 EXT REG LOGIC VIN GND VOUT

Commit message: Fix PCB DRC: power trace width and silkscreen overlap
Parts:
- added J4_ALT: BATTERY_ALT_2P_2.54, Connector_PinHeader_2.54mm:PinHeader_1x02_P2.54mm_Vertical, B.Cu at (82.0, 66.0)
Connections:
- JP1 pad 3: (no net) -> VBAT_SW
- U1 pad 1: GPIO5_SPARE -> GPIO5
- U2 pad 12: GPIO20_SPARE -> GPIO5
Routing:
- net GPIO20_SPARE: track 114.5 -> 2.54 mm
- net GPIO5: track 0.00 -> 87.4 mm
- net GND: track 167.6 -> 172.6 mm
- net VBAT_SW: track 194.9 -> 199.0 mm
- net GPIO5_SPARE: track 2.54 -> 0.00 mm
Other:
- outline, holes or cut-outs redrawn
- board text added: "1S"
- board text added: "1S/3.5-4.2V"
- board text added: "2S"
- board text added: "2S/5VREG"
- board text added: "G5/SLEEP"
- board text removed: "1S/3.7V"
- board text removed: "2S/7.4V"
- board text removed: "G5"
- board text removed: "Online"
