File: electronics/kicad/hsd-antweight-2s-v4/hsd-antweight-2s-v4.kicad_pcb (KiCad board)
At the start: 2 copper layers, 78 x 56 mm, 11 parts, among them J10 5V(3.7-5V) GND VLIPO, J4 BATTERY, J4_ALT BATTERY_ALT_2P_2.54, J5 MOTOR LEFT, J6 MOTOR RIGHT, SW1 SW EXT VBAT_RAW/VBAT_SW, U1 ESP32-C3 SUPERMINI, U2 DRV8833, U3 EXT REG LOGIC VIN GND VOUT

Commit message: kicad(v4): refresh renders and PCBWay production package
Other:
- board text added: "Ant-weight robot controller v4"
- board text added: "Design by Rein"
- board text added: "HACKERSPACE DRENTHE"
- board text added: "HSD-ANTWEIGHT-2S-v4 20260827"
- board text added: "Idea by Wallie"
- board text added: "Online"
- board text added: "ROBOKTOBER"
- board text removed: "HSD-ANTWEIGHT-2S-v4"
