File: electronics/kicad/hsd-antweight-2s-v4/hsd-antweight-2s-v4.kicad_pcb (KiCad board)
At the start: 2 copper layers, 78 x 56 mm, 11 parts, among them J10 5V(3.7-5V) GND VLIPO, J4 BATTERY, J4_ALT BATTERY_ALT_2P_2.54, J5 MOTOR LEFT, J6 MOTOR RIGHT, SW1 SW EXT VBAT_RAW/VBAT_SW, U1 ESP32-C3 SUPERMINI, U2 DRV8833, U3 EXT REG LOGIC VIN GND VOUT

Commit message: Update V4 PCBWay production files after logo update
Other:
- board text added: "This PCB is manufactured"
- board text added: "and sponsored by:"
